Commit message: Update: Improved Isaac Sim integration, added gripper, new launch files and docs

File: src/DOBOT_6Axis_ROS2_V4/cra_description/urdf/cr20_robot.urdf (robot description, URDF)
Before this commit: robot cr20_robot, 8 links, 7 joints
Links:
- removed link world
- added link gripper_link, mass 0.5; collision mesh filename=/home/iudc/dobot_ws/src/DOBOT_6Axis_ROS2_V4/cra_description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; visual mesh filename=/home/iudc/dobot_ws/src/DOBOT_6Axis_ROS2_V4/cra_description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
- link Link1: geometry collision mesh filename=/home/iudc/dobot_ws/src/DOBOT_6Axis_ROS2_V4/cra_description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; visual mesh filename=/home/iudc/dobot_ws/src/DOBOT_6Axis_ROS2_V4/cra_description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
- link Link2: geometry collision mesh filename=/home/iudc/dobot_ws/src/DOBOT_6Axis_ROS2_V4/cra_description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; visual mesh filename=/home/iudc/dobot_ws/src/DOBOT_6Axis_ROS2_V4/cra_description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
- link Link3: geometry collision mesh filename=/home/iudc/dobot_ws/src/DOBOT_6Axis_ROS2_V4/cra_description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; visual mesh filename=/home/iudc/dobot_ws/src/DOBOT_6Axis_ROS2_V4/cra_description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
- link Link4: geometry collision mesh filename=/home/iudc/dobot_ws/src/DOBOT_6Axis_ROS2_V4/cra_description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; visual mesh filename=/home/iudc/dobot_ws/src/DOBOT_6Axis_ROS2_V4/cra_description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
- link Link5: geometry collision mesh filename=/home/iudc/dobot_ws/src/DOBOT_6Axis_ROS2_V4/cra_description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; visual mesh filename=/home/iudc/dobot_ws/src/DOBOT_6Axis_ROS2_V4/cra_description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
- link Link6: geometry collision mesh filename=/home/iudc/dobot_ws/src/DOBOT_6Axis_ROS2_V4/cra_description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; visual mesh filename=/home/iudc/dobot_ws/src/DOBOT_6Axis_ROS2_V4/cra_description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
- link base_link: geometry collision mesh filename=/home/iudc/dobot_ws/src/DOBOT_6Axis_ROS2_V4/cra_description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; visual mesh filename=/home/iudc/dobot_ws/src/DOBOT_6Axis_ROS2_V4/cra_description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
Joints:
- removed joint world_joint
- added joint gripper_joint: type fixed, parent Link6, child gripper_link, origin xyz=0 0 0 rpy=0 0 0
- joint joint1: limit lower=-6.28 upper=6.28 effort=150.0 velocity=3.14 -> lower=-6.28 upper=6.28 effort=150 velocity=3.14
- joint joint2: limit lower=-6.28 upper=6.28 effort=150.0 velocity=3.14 -> lower=-6.28 upper=6.28 effort=150 velocity=3.14
- joint joint3: limit lower=-2.9 upper=2.9 effort=150.0 velocity=3.14 -> lower=-2.9 upper=2.9 effort=150 velocity=3.14
- joint joint4: limit lower=-6.28 upper=6.28 effort=50.0 velocity=3.14 -> lower=-6.28 upper=6.28 effort=50 velocity=3.14
- joint joint5: limit lower=-6.28 upper=6.28 effort=50.0 velocity=3.14 -> lower=-6.28 upper=6.28 effort=50 velocity=3.14
- joint joint6: limit lower=-6.28 upper=6.28 effort=50.0 velocity=3.14 -> lower=-6.28 upper=6.28 effort=50 velocity=3.14
